File: hardware/pod_basic_expander_2.kicad_pcb (KiCad board)
At the start: 2 copper layers, 45 x 44 mm, 7 parts, among them J1 POD, SW1 SW_Push, SW2 SW_Push, SW3 SW_Push, SW4 SW_Push

Commit message: PCB changes
Other:
- board text removed: "KnightHill Engineering"
Changed lines of the file:
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@@
   (gr_circle (center 76 69) (end 77 70)
     (stroke (width 0.05) (type default)) (fill none) (layer "Edge.Cuts"))
-  (gr_text "KnightHill Engineering\n" (at 90 70) (layer "F.SilkS")
-    (effects (font (size 1 1) (thickness 0.1)) (justify left bottom))
-  )
   (segment (start 107 91) (end 108.7 92.7) (width 0.2) (layer "B.Cu") (net 5))
   (segment (start 107 87) (end 107 91) (width 0.2) (layer "B.Cu") (net 5))
