File: hardware/pod_basic_expander.kicad_pcb (KiCad board)
At the start: 2 copper layers, 45 x 44 mm, 7 parts, among them J1 POD, SW1 SW_Push, SW2 SW_Push, SW3 SW_Push, SW4 SW_Push

Commit message: pcb changes
Other:
- outline, holes or cut-outs redrawn
Changed lines of the file:
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@@
       (plot_on_all_layers_selection 0x0000000_00000000)
       (disableapertmacros false)
-      (usegerberextensions false)
-      (usegerberattributes true)
-      (usegerberadvancedattributes true)
-      (creategerberjobfile true)
+      (usegerberextensions true)
+      (usegerberattributes false)
+      (usegerberadvancedattributes false)
+      (creategerberjobfile false)
       (dashed_line_dash_ratio 12.000000)
       (dashed_line_gap_ratio 3.000000)
@@
       (psa4output false)
       (plotreference true)
-      (plotvalue true)
+      (plotvalue false)
       (plotinvisibletext false)
       (sketchpadsonfab false)
-      (subtractmaskfromsilk false)
+      (subtractmaskfromsilk true)
       (outputformat 1)
       (mirror false)
-      (drillshape 1)
+      (drillshape 0)
       (scaleselection 1)
-      (outputdirectory "")
+      (outputdirectory "/home/bojidar/gerber/")
     )
   )
@@
   (gr_circle (center 63 81) (end 64 82)
     (stroke (width 0.05) (type default)) (fill none) (layer "Edge.Cuts"))
-  (gr_rect (start 60 40) (end 105 84)
-    (stroke (width 0.05) (type default)) (fill none) (layer "Edge.Cuts"))
+  (gr_line (start 60 41) (end 60 82.5)
+    (stroke (width 0.05) (type default)) (layer "Edge.Cuts"))
+  (gr_arc (start 61.5 84) (mid 60.43934 83.56066) (end 60 82.5)
+    (stroke (width 0.05) (type default)) (layer "Edge.Cuts"))
+  (gr_line (start 61.5 84) (end 103.5 84)
+    (stroke (width 0.05) (type default)) (layer "Edge.Cuts"))
+  (gr_line (start 105 41) (end 105 82.5)
+    (stroke (width 0.05) (type default)) (layer "Edge.Cuts"))
+  (gr_arc (start 60 41) (mid 60.292893 40.292893) (end 61 40)
+    (stroke (width 0.05) (type default)) (layer "Edge.Cuts"))
   (gr_circle (center 102 43) (end 103 44)
     (stroke (width 0.05) (type default)) (fill none) (layer "Edge.Cuts"))
+  (gr_arc (start 105 82.5) (mid 104.56066 83.56066) (end 103.5 84)
+    (stroke (width 0.05) (type default)) (layer "Edge.Cuts"))
   (gr_circle (center 102 81) (end 103 82)
     (stroke (width 0.05) (type default)) (fill none) (layer "Edge.Cuts"))
+  (gr_line (start 61 40) (end 104 40)
+    (stroke (width 0.05) (type default)) (layer "Edge.Cuts"))
   (gr_circle (center 63 43) (end 64 44)
     (stroke (width 0.05) (type default)) (fill none) (layer "Edge.Cuts"))
+  (gr_arc (start 104 40) (mid 104.707107 40.292893) (end 105 41)
+    (stroke (width 0.05) (type default)) (layer "Edge.Cuts"))
   (gr_text "KnightHill Engineering\nE/S Pod expander V1\n" (at 86 45) (layer "F.SilkS")
     (effects (font (size 1 1) (thickness 0.1)) (justify bottom))
   )
-  (segment (start 94 65) (end 95.7 66.7) (width 0.2) (layer "B.Cu") (net 5))
-  (segment (start 94 61) (end 94 65) (width 0.2) (layer "B.Cu") (net 5))
+  (segment (start 93 64) (end 95.7 66.7) (width 0.2) (layer "B.Cu") (net 5))
+  (segment (start 79.5 55.2) (end 88.2 55.2) (width 0.2) (layer "B.Cu") (net 5))
+  (segment (start 93 60) (end 93 64) (width 0.2) (layer "B.Cu") (net 5))
+  (segment (start 88.2 55.2) (end 93 60) (width 0.2) (layer "B.Cu") (net 5))
   (segment (start 95.7 66.7) (end 97.1 66.7) (width 0.2) (layer "B.Cu") (net 5))
-  (segment (start 88.2 55.2) (end 94 61) (width 0.2) (layer "B.Cu") (net 5))
-  (segment (start 79.5 55.2) (end 88.2 55.2) (width 0.2) (layer "B.Cu") (net 5))
   (segment (start 97.1 64.16) (end 93.84 64.16) (width 0.2) (layer "F.Cu") (net 6))
   (segment (start 93.84 64.16) (end 88.93 69.07) (width 0.2) (layer "F.Cu") (net 6))
@@
       )
     )
-  )
-  (zone (net 0) (net_name "") (layer "F.Cu") (hatch edge 0.5)
-    (connect_pads (clearance 0))
-    (min_thickness 0.25) (filled_areas_thickness no)
-    (keepout (tracks allowed) (vias allowed) (pads allowed) (copperpour not_allowed) (footprints allowed))
-    (fill (thermal_gap 0.5) (thermal_bridge_width 0.5))
-    (polygon
-      (pts
-        (xy 92.989194 46.56256)
-        (xy 93 63)
-        (xy 99 63)
-        (xy 98.989194 46.56256)
-      )
-    )
