File: hardware/basic_expander_v2.1/basic_expander_v2.1.kicad_pcb (KiCad board)
At the start: 2 copper layers, 45 x 58 mm, 13 parts, among them J1 POD, SW1 SW_Push, SW2 SW_Push, SW3 SW_Push, SW4 SW_Push, SW5 SW_Push, SW6 SW_Push

Commit message: fix pots orientation
Parts:
- moved RV2 13.3 mm to (82.7, 71.7), turned to 0 degrees
- moved RV1 12.1 mm to (82.7, 55.0), turned to 0 degrees
Connections:
- RV1 pad 1: VDDA -> GND
- RV1 pad 3: GND -> VDDA
- RV2 pad 1: VDDA -> GND
- RV2 pad 3: GND -> VDDA
Routing:
- net /A1/D16: track 10.2 -> 19.2 mm
- net /A7/D22: track 14.3 -> 20.3 mm
Changed lines of the file:
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@@
   (net 12 "/D7")
   (footprint "Potentiometer_THT:Potentiometer_Alpha_RD901F-40-00D_Single_Vertical" (layer "F.Cu")
-    (at 93.6 79.3 180)
+    (at 82.7 71.7)
     (descr "Potentiometer, vertical, 9mm, single, http://www.taiwanalpha.com.tw/downloads?target=products&id=113")
     (tags "potentiometer vertical 9mm single")
@@
     (property "ki_keywords" "resistor variable")
     (attr through_hole)
-    (fp_text reference "RV2" (at 7.85 10.55) (layer "F.SilkS")
+    (fp_text reference "RV2" (at 7.4 -5.1) (layer "F.SilkS")
         (effects (font (size 1 1) (thickness 0.15)))
     )
@@
     (fp_circle (center 7.5 2.5) (end 7.5 -1)
       (stroke (width 0.1) (type solid)) (fill none) (layer "F.Fab"))
-    (pad "" thru_hole oval (at 7.5 -2.3 270) (size 2.72 3.24) (drill oval 1.1 1.8) (layers "*.Cu" "*.Mask"))
-    (pad "" thru_hole oval (at 7.5 7.3 270) (size 2.72 3.24) (drill oval 1.1 1.8) (layers "*.Cu" "*.Mask"))
-    (pad "1" thru_hole rect (at 0 0 270) (size 1.8 1.8) (drill 1) (layers "*.Cu" "*.Mask")
-      (net 4 "VDDA") (pinfunction "1") (pintype "passive"))
-    (pad "2" thru_hole circle (at 0 2.5 270) (size 1.8 1.8) (drill 1) (layers "*.Cu" "*.Mask")
+    (pad "" thru_hole oval (at 7.5 -2.3 90) (size 2.72 3.24) (drill oval 1.1 1.8) (layers "*.Cu" "*.Mask"))
+    (pad "" thru_hole oval (at 7.5 7.3 90) (size 2.72 3.24) (drill oval 1.1 1.8) (layers "*.Cu" "*.Mask"))
+    (pad "1" thru_hole rect (at 0 0 90) (size 1.8 1.8) (drill 1) (layers "*.Cu" "*.Mask")
+      (net 1 "GND") (pinfunction "1") (pintype "passive"))
+    (pad "2" thru_hole circle (at 0 2.5 90) (size 1.8 1.8) (drill 1) (layers "*.Cu" "*.Mask")
       (net 6 "/A7{slash}D22") (pinfunction "2") (pintype "passive"))
-    (pad "3" thru_hole circle (at 0 5 270) (size 1.8 1.8) (drill 1) (layers "*.Cu" "*.Mask")
-      (net 1 "GND") (pinfunction "3") (pintype "passive"))
+    (pad "3" thru_hole circle (at 0 5 90) (size 1.8 1.8) (drill 1) (layers "*.Cu" "*.Mask")
+      (net 4 "VDDA") (pinfunction "3") (pintype "passive"))
     (model "${KICAD6_3DMODEL_DIR}/Potentiometer_THT.3dshapes/Potentiometer_Alpha_RD901F-40-00D_Single_Vertical.wrl"
       (offset (xyz 0 0 0))
@@
   )
   (footprint "Potentiometer_THT:Potentiometer_Alpha_RD901F-40-00D_Single_Vertical" (layer "F.Cu")
-    (at 93.6 60.3 180)
+    (at 82.7 55)
     (descr "Potentiometer, vertical, 9mm, single, http://www.taiwanalpha.com.tw/downloads?target=products&id=113")
     (tags "potentiometer vertical 9mm single")
@@
     (property "ki_keywords" "resistor variable")
     (attr through_hole)
-    (fp_text reference "RV1" (at 7.6 10.8) (layer "F.SilkS")
+    (fp_text reference "RV1" (at 7.5 -5.2) (layer "F.SilkS")
         (effects (font (size 1 1) (thickness 0.15)))
     )
@@
     (fp_circle (center 7.5 2.5) (end 7.5 -1)
       (stroke (width 0.1) (type solid)) (fill none) (layer "F.Fab"))
-    (pad "" thru_hole oval (at 7.5 -2.3 270) (size 2.72 3.24) (drill oval 1.1 1.8) (layers "*.Cu" "*.Mask"))
-    (pad "" thru_hole oval (at 7.5 7.3 270) (size 2.72 3.24) (drill oval 1.1 1.8) (layers "*.Cu" "*.Mask"))
-    (pad "1" thru_hole rect (at 0 0 270) (size 1.8 1.8) (drill 1) (layers "*.Cu" "*.Mask")
-      (net 4 "VDDA") (pinfunction "1") (pintype "passive"))
-    (pad "2" thru_hole circle (at 0 2.5 270) (size 1.8 1.8) (drill 1) (layers "*.Cu" "*.Mask")
+    (pad "" thru_hole oval (at 7.5 -2.3 90) (size 2.72 3.24) (drill oval 1.1 1.8) (layers "*.Cu" "*.Mask"))
+    (pad "" thru_hole oval (at 7.5 7.3 90) (size 2.72 3.24) (drill oval 1.1 1.8) (layers "*.Cu" "*.Mask"))
+    (pad "1" thru_hole rect (at 0 0 90) (size 1.8 1.8) (drill 1) (layers "*.Cu" "*.Mask")
+      (net 1 "GND") (pinfunction "1") (pintype "passive"))
+    (pad "2" thru_hole circle (at 0 2.5 90) (size 1.8 1.8) (drill 1) (layers "*.Cu" "*.Mask")
       (net 5 "/A1{slash}D16") (pinfunction "2") (pintype "passive"))
-    (pad "3" thru_hole circle (at 0 5 270) (size 1.8 1.8) (drill 1) (layers "*.Cu" "*.Mask")
-      (net 1 "GND") (pinfunction "3") (pintype "passive"))
+    (pad "3" thru_hole circle (at 0 5 90) (size 1.8 1.8) (drill 1) (layers "*.Cu" "*.Mask")
+      (net 4 "VDDA") (pinfunction "3") (pintype "passive"))
     (model "${KICAD6_3DMODEL_DIR}/Potentiometer_THT.3dshapes/Potentiometer_Alpha_RD901F-40-00D_Single_Vertical.wrl"
       (offset (xyz 0 0 0))
@@
     (effects (font (size 1 1) (thickness 0.1)) (justify bottom))
   )
-  (segment (start 95.55 57.8) (end 96 58.25) (width 0.2) (layer "F.Cu") (net 5))
-  (segment (start 97.58 63.33) (end 99.5 63.33) (width 0.2) (layer "F.Cu") (net 5))
-  (segment (start 96 61.75) (end 97.58 63.33) (width 0.2) (layer "F.Cu") (net 5))
-  (segment (start 93.6 57.8) (end 95.55 57.8) (width 0.2) (layer "F.Cu") (net 5))
-  (segment (start 96 58.25) (end 96 61.75) (width 0.2) (layer "F.Cu") (net 5))
-  (segment (start 93.6 76.8) (end 96.25 74.15) (width 0.2) (layer "F.Cu") (net 6))
-  (segment (start 96.25 67.5) (end 97.88 65.87) (width 0.2) (layer "F.Cu") (net 6))
-  (segment (start 97.88 65.87) (end 99.5 65.87) (width 0.2) (layer "F.Cu") (net 6))
-  (segment (start 96.25 74.15) (end 96.25 67.5) (width 0.2) (layer "F.Cu") (net 6))
+  (segment (start 93.67 57.5) (end 99.5 63.33) (width 0.2) (layer "F.Cu") (net 5))
+  (segment (start 82.7 57.5) (end 93.67 57.5) (width 0.2) (layer "F.Cu") (net 5))
+  (segment (start 82.7 74.2) (end 91.17 74.2) (width 0.2) (layer "F.Cu") (net 6))
+  (segment (start 91.17 74.2) (end 99.5 65.87) (width 0.2) (layer "F.Cu") (net 6))
   (segment (start 100.65 71.534314) (end 100.65 69.56) (width 0.2) (layer "F.Cu") (net 7))
   (segment (start 102.25 77.082942) (end 101.45 76.282942) (width 0.2) (layer "F.Cu") (net 7))

Commit message: add v2.1 gerber files
Parts:
- RV1, RV2: footprint Potentiometer_THT:Potentiometer_Alpha_RD901F-40-00D_Single_Vertical -> Local:Potentiometer_uxcel_9mm_Single_Vertical
Changed lines of the file:
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@@
       (drillshape 0)
       (scaleselection 1)
-      (outputdirectory "/home/bojidar/src/daisy/khill/BasicExpander/hardware/DrillMapFiles/")
+      (outputdirectory "GerberFiles/")
     )
   )
@@
   (net 11 "/D8")
   (net 12 "/D7")
-  (footprint "Potentiometer_THT:Potentiometer_Alpha_RD901F-40-00D_Single_Vertical" (layer "F.Cu")
+  (footprint "Local:Potentiometer_uxcel_9mm_Single_Vertical" (layer "F.Cu")
     (at 82.7 71.7)
     (descr "Potentiometer, vertical, 9mm, single, http://www.taiwanalpha.com.tw/downloads?target=products&id=113")
@@
     (property "ki_keywords" "resistor variable")
     (attr through_hole)
-    (fp_text reference "RV2" (at 7.4 -5.1) (layer "F.SilkS")
-        (effects (font (size 1 1) (thickness 0.15)))
-    )
-    (fp_text value "10k" (at 2.5 6.43) (layer "F.Fab")
-        (effects (font (size 1 1) (thickness 0.15)))
-    )
-    (fp_text user "${REFERENCE}" (at 7.5 2.5) (layer "F.Fab")
+    (fp_text reference "RV2" (at 6.71 -4.64 180) (layer "F.SilkS")
+        (effects (font (size 1 1) (thickness 0.15)))
+    )
+    (fp_text value "10k" (at 7.366 10.922 180) (layer "F.Fab")
+        (effects (font (size 1 1) (thickness 0.15)))
+    )
+    (fp_text user "${REFERENCE}" (at 7.62 2.54) (layer "F.Fab")
         (effects (font (size 1 1) (thickness 0.15)))
     )
@@
     (fp_circle (center 7.5 2.5) (end 7.5 -1)
       (stroke (width 0.1) (type solid)) (fill none) (layer "F.Fab"))
-    (pad "" thru_hole oval (at 7.5 -2.3 90) (size 2.72 3.24) (drill oval 1.1 1.8) (layers "*.Cu" "*.Mask"))
-    (pad "" thru_hole oval (at 7.5 7.3 90) (size 2.72 3.24) (drill oval 1.1 1.8) (layers "*.Cu" "*.Mask"))
+    (pad "" thru_hole oval (at 7.5 -2.3 90) (size 2.72 3.58) (drill oval 1.1 2.2) (layers "*.Cu" "*.Mask"))
+    (pad "" thru_hole oval (at 7.5 7.3 90) (size 2.696 3.58) (drill oval 1.1 2.2 (offset 0.012 0.012)) (layers "*.Cu" "*.Mask"))
     (pad "1" thru_hole rect (at 0 0 90) (size 1.8 1.8) (drill 1) (layers "*.Cu" "*.Mask")
       (net 1 "GND") (pinfunction "1") (pintype "passive"))
@@
     (pad "" np_thru_hole circle (at 0 0 90) (size 2.2 2.2) (drill 2.2) (layers "*.Cu" "*.Mask"))
   )
-  (footprint "Potentiometer_THT:Potentiometer_Alpha_RD901F-40-00D_Single_Vertical" (layer "F.Cu")
+  (footprint "Local:Potentiometer_uxcel_9mm_Single_Vertical" (layer "F.Cu")
     (at 82.7 55)
     (descr "Potentiometer, vertical, 9mm, single, http://www.taiwanalpha.com.tw/downloads?target=products&id=113")
@@
     (property "ki_keywords" "resistor variable")
     (attr through_hole)
-    (fp_text reference "RV1" (at 7.5 -5.2) (layer "F.SilkS")
-        (effects (font (size 1 1) (thickness 0.15)))
-    )
-    (fp_text value "10k" (at 2.5 -0.7) (layer "F.Fab")
+    (fp_text reference "RV1" (at 6.71 -4.64 180) (layer "F.SilkS")
+        (effects (font (size 1 1) (thickness 0.15)))
+    )
+    (fp_text value "10k" (at 7.366 10.922 180) (layer "F.Fab")
         (effects (font (size 1 1) (thickness 0.15)))
     )
@@
     (fp_circle (center 7.5 2.5) (end 7.5 -1)
       (stroke (width 0.1) (type solid)) (fill none) (layer "F.Fab"))
-    (pad "" thru_hole oval (at 7.5 -2.3 90) (size 2.72 3.24) (drill oval 1.1 1.8) (layers "*.Cu" "*.Mask"))
-    (pad "" thru_hole oval (at 7.5 7.3 90) (size 2.72 3.24) (drill oval 1.1 1.8) (layers "*.Cu" "*.Mask"))
+    (pad "" thru_hole oval (at 7.5 -2.3 90) (size 2.72 3.58) (drill oval 1.1 2.2) (layers "*.Cu" "*.Mask"))
+    (pad "" thru_hole oval (at 7.5 7.3 90) (size 2.696 3.58) (drill oval 1.1 2.2 (offset 0.012 0.012)) (layers "*.Cu" "*.Mask"))
     (pad "1" thru_hole rect (at 0 0 90) (size 1.8 1.8) (drill 1) (layers "*.Cu" "*.Mask")
       (net 1 "GND") (pinfunction "1") (pintype "passive"))
