File: hardware/basic_expander_v2.1/basic_expander_v2.1.kicad_sch (KiCad schematic)
At the start: 13 parts, among them J1 POD, SW1 SW_Push, SW2 SW_Push, SW3 SW_Push, SW4 SW_Push, SW5 SW_Push, SW6 SW_Push

Commit message: fix pots orientation
Connections:
- net GND: now also RV1.1, RV2.1; no longer RV1.3, RV2.3
- net VDDA: now also RV1.3, RV2.3; no longer RV1.1, RV2.1
Other:
- moved on the sheet: RV2, SW1, SW2, SW3, SW4, SW5, SW6

Commit message: add v2.1 gerber files
Parts:
- RV1, RV2: footprint Potentiometer_THT:Potentiometer_Alpha_RD901F-40-00D_Single_Vertical -> Local:Potentiometer_uxcel_9mm_Single_Vertical
Other:
- moved on the sheet: J1, RV1, RV2, SW1, SW2, SW3, SW4, SW5, SW6
