File: hardware/basic_expander_v3/basic_expander_v3.kicad_sch (KiCad schematic)
At the start: 27 parts, among them J1 Daisy Pod, SW1 SW_Push, SW2 SW_Push, SW3 SW_Push, SW4 SW_Push, SW5 SW_Push, SW6 SW_Push, SW7 SW_Push, SW8 SW_Push, U1 4051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

Commit message: add 4 pots
Parts:
- added RV5, RV6, RV7, RV8: 10k, Potentiometer_THT:Potentiometer_Alpha_RD901F-40-00D_Single_Vertical, symbol Device:R_Potentiometer_US
Connections:
- net GND: now also RV5.1, RV6.1, RV7.1, RV8.1
- net RV1: now also U1.1 (X4); no longer U1.13 (X0)
- net RV2: now also U1.5 (X5); no longer U1.14 (X1)
- net RV3: now also U1.2 (X6); no longer U1.15 (X2)
- net RV4: now also U1.4 (X7); no longer U1.12 (X3)
- net VDDA: now also RV5.3, RV6.3, RV7.3, RV8.3
- new net RV5: RV5.2, U1.12 (X3)
- new net RV6: RV6.2, U1.13 (X0)
- new net RV7: RV7.2, U1.14 (X1)
- new net RV8: RV8.2, U1.15 (X2)
- no-connect marks 11 -> 7
Other:
- moved on the sheet: RV1, RV2, RV3, RV4
